File: PCB/Mike-ky-board.kicad_pcb (KiCad board)
At the start: 2 copper layers, 1008.5 x 98.7 mm, 190 parts, among them SW100 SW_Push_45deg, SW101 SW_Push_45deg, SW102 RotaryEncoder_Switch_MP, SW109 SW_Push_45deg, SW112 SW_Push_45deg, SW113 SW_Push_45deg, SW114 SW_Push_45deg, SW115 SW_Push_45deg, SW116 SW_Push_45deg, SW117 SW_Push_45deg, SW118 SW_Push_45deg, SW119 SW_Push_45deg, SW120 SW_Push_45deg, SW121 SW_Push_45deg, SW122 SW_Push_45deg, SW123 SW_Push_45deg, SW124 SW_Push_45deg, SW125 SW_Push_45deg, SW126 SW_Push_45deg, SW127 SW_Push_45deg, SW128 SW_Push_45deg, SW129 SW_Push_45deg, SW130 SW_Push_45deg, SW131 SW_Push_45deg, SW132 SW_Push_45deg, SW133 SW_Push_45deg, SW134 SW_Push_45deg, SW135 SW_Push_45deg, SW136 SW_Push_45deg, SW137 SW_Push_45deg, SW138 SW_Push_45deg, SW139 SW_Push_45deg, SW140 SW_Push_45deg, SW141 SW_Push_45deg, SW142 SW_Push_45deg, SW143 SW_Push_45deg, SW144 SW_Push_45deg, SW145 SW_Push_45deg, SW146 SW_Push_45deg, SW147 SW_Push_45deg, SW148 SW_Push_45deg, SW149 SW_Push_45deg, SW150 SW_Push_45deg, SW151 SW_Push_45deg, SW152 SW_Push_45deg, SW153 SW_Push_45deg, SW154 SW_Push_45deg, SW155 SW_Push_45deg, SW156 SW_Push_45deg, SW157 SW_Push_45deg, SW158 SW_Push_45deg, SW159 SW_Push_45deg, SW160 SW_Push_45deg, SW161 SW_Push_45deg, SW162 SW_Push_45deg, SW163 SW_Push_45deg, SW164 SW_Push_45deg, SW165 SW_Push_45deg, SW166 SW_Push_45deg, SW167 SW_Push_45deg, SW168 SW_Push_45deg, SW169 SW_Push_45deg, SW170 SW_Push_45deg, SW171 SW_Push_45deg, SW172 SW_Push_45deg, SW173 SW_Push_45deg, SW174 SW_Push_45deg, SW175 SW_Push_45deg, SW176 SW_Push_45deg, SW177 SW_Push_45deg, SW178 SW_Push_45deg, SW179 SW_Push_45deg, SW180 SW_Push_45deg, SW181 SW_Push_45deg, SW182 SW_Push_45deg, SW82 RotaryEncoder_Switch_MP, SW83 SW_Push_45deg, SW84 SW_DIP_x01, SW85 SW_Push_45deg, SW86 SW_Push_45deg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

Commit message: l
Routing:
- net /Matrix/Col7: track 1004.1 -> 964.7 mm
